File: Hardware/TILDO/TI_HV_LDO.kicad_pcb (KiCad board)
At the start: 2 copper layers, 36 x 15 mm, 10 parts, among them J1 Conn_01x02, J2 Conn_01x02, J3 Conn_01x02, U1 TPS7A19

Commit message: More updates before ordering.
Parts:
- C1: footprint Capacitors_SMD:CP_Elec_6.3x4.5 -> Capacitors_SMD:C_1210_HandSoldering
- moved J2 12.3 mm to (143.2, 101.0), turned to 270 degrees
- moved J1 9.62 mm to (141.5, 89.5), turned to 90 degrees
- moved J3 8.96 mm to (152.8, 101.0), turned to 90 degrees
- moved C1 2.50 mm to (141.5, 95.0)
- moved R1 1.30 mm to (148.6, 100.0)
Routing:
- net Net-(C3-Pad1): track 10.9 -> 3.25 mm
- net Net-(J2-Pad1): track 15.2 -> 10.0 mm
Other:
- board size 36 x 15 mm -> 30 x 16 mm
